File: Partie_Informatique/Eagle/Project/ESP_LoRa_GSM.brd (EAGLE design)
At the start: 90 x 58 mm, 33 parts, among them J1 U.FL, Q1 Si2305, Q2 BSS131, Q6 PT17-21C, U1 ESP-WROOM-03, U2 BK7000-V2, U3 WIRELESS-LORA-RFM95W#SMD

Commit message: Seance18
Ajout dernière version du projet EAGLE.
Parts:
- added C7: 100n, eagle-ltspice:C1206
- added C8: 10u, eagle-ltspice:C1206
- added Q3: Si2305, transistor-small-signal:SOT23
- added Q4: BSS131, transistor-small-signal:SOT23
- added R5, R6: 100k, eagle-ltspice:R1206
- moved Q6 50.5 mm to (84.8, 47.8)
- moved R22 44.8 mm to (84.3, 44.9), turned to 180 degrees
- moved R21 41.0 mm to (32.1, 12.4), turned to 270 degrees
- moved LED_G 39.0 mm to (61.9, 14.7), turned to 270 degrees
- moved JP3 38.7 mm to (36.5, 13.8), turned to 270 degrees
- moved R25 38.5 mm to (57.5, 13.3), turned to 180 degrees
- moved R23 36.4 mm to (57.5, 18.3), turned to 180 degrees
- moved LED_R 36.1 mm to (61.9, 19.8), turned to 270 degrees
- moved SJ1 21.8 mm to (31.4, 34.8), flipped to the bottom, turned to 270 degrees
- moved R4 12.6 mm to (55.1, 52.2), turned to 270 degrees
- moved R2 8.33 mm to (81.9, 38.7)
- moved Q2 7.26 mm to (51.6, 52.2), turned to 90 degrees
- moved RST 5.52 mm to (80.6, 8.41), turned to 90 degrees
- moved C4 4.76 mm to (58.7, 46.8)
- moved C3 4.47 mm to (77.9, 37.8), turned to 270 degrees
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Connections:
- removed net DIO: SJ1.2, U1.11
- removed net N$7: LED_R.A, R23.2
- removed net N$8: LED_G.A, R25.2
- new net BUSY: U1.9, U3.B1
- new net DIO1: SJ1.3, U3.B2
- new net N$2: SJ1.2, U1.8
- new net N$3: LED_R.C, R23.1
- new net N$4: LED_G.C, R25.1
- new net N$9: Q3.1, Q4.3, R5.1
- new net PERIF: Q4.1, R6.2, U1.11
- new net V+: C7.1, C8.1, D1.1, JP3.3, Q3.3, Q6.2, R21.2
- net CMD_ALIM(SIM): now also U1.6; no longer U1.23
- net DHT: now also U1.32; no longer U1.8
- net DIO3: now also U1.14; no longer SJ1.3
- net EXT1: now also U1.13; no longer U1.14
- net EXT2: now also U1.7; no longer U1.32
- net GND: now also C7.2, C8.2, Q4.2, R23.2, R25.2, R6.1; no longer LED_G.C, LED_R.C
- net IOPWRKEY(SIM): now also U1.26; no longer U1.12
- net IOSLEEP(SIM): now also U1.10; no longer U1.16
- net LED_G: now also LED_G.A, U1.24; no longer R25.1, U1.10
- net LED_R: now also LED_R.A, U1.16; no longer R23.1, U1.9
- net LIGHT: now also U1.5
- net RFM_RST: now also U1.12; no longer U1.13
- net VCC: now also Q3.2, R5.2; no longer D1.1, JP3.3, Q6.2, R21.2
Routing:
- net GND: track 283.2 -> 48.9 mm, vias 11 -> 67
- net V+: track 0.00 -> 94.3 mm, vias 0 -> 2
- net BUSY: track 0.00 -> 49.8 mm, vias 0 -> 2
- net N$2: track 0.00 -> 46.3 mm, vias 0 -> 1
- net VCC: track 190.3 -> 155.6 mm, vias 4 -> 10
- net EXT2: track 87.1 -> 54.9 mm, vias 2 -> 1
- net DIO: track 27.5 -> 0.00 mm, vias 2 -> 0
- net DIO0: track 32.0 -> 4.89 mm, vias 2 -> 1
- net IOPWRKEY(SIM): track 29.1 -> 54.9 mm, vias 2 -> 1
- net LIGHT: track 3.41 -> 28.7 mm, vias 0 -> 2
- net MOSI: track 80.3 -> 66.4 mm
- net SDA: track 91.3 -> 78.7 mm, vias 5 -> 2
- net MISO: track 43.1 -> 54.9 mm
- net LED_G: track 15.3 -> 4.02 mm, vias 2 -> 0
- net SCL: track 85.3 -> 74.6 mm, vias 3 -> 2
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Other:
- board text added: "DIO1"
- board text added: "GND DHT V+"
- board text added: "GND Ext1 Ext2 VBAT"
- board text added: "LoRa GSM Xavier MIRRIONE Daniel CEBAN"
- board text added: "VCC SCL SDA GND"
- board text removed: "(users.polytech.unice.fr/~ferrero/recherche.html)"
- board text removed: "A1"
- board text removed: "A6"
- board text removed: "B2"
- board text removed: "DIO3"
- board text removed: "DRDY1 gnd"
- board text removed: "E+ red A/B- white A/B+ blue/green E- black"
- board text removed: "LoRa Bee Scale V1.61 Christian.PETER @univ-cotedazur.fr"
- board text removed: "SDA SCL gnd V+"
- board text removed: "Short SJ7 if U4 used"
- board text removed: "V+ DHT GND"
- board text removed: "V+ GND SCL SDA"
- board text removed: "V1.61"
- board text removed: "http://rucher.polytech.unice.fr"
- board text removed: "with external antenna connected on J1, cut here"
