File: Partie_Informatique/Eagle/Project/ESP_LoRa_GSM.sch (EAGLE design)
At the start: 34 parts, among them J1 U.FL, Q1 Si2305, Q2 BSS131, Q6 PT17-21C, U1 ESP-WROOM-03, U2 BK7000-V2, U3 WIRELESS-LORA-RFM95W#SMD

Commit message: Seance18
Ajout dernière version du projet EAGLE.
Parts:
- removed JP5(SIM7000): (no value), pinhead:PINHD-1X7
- added C7: 100n, eagle-ltspice:CC1206
- added C8: 10u, eagle-ltspice:CC1206
- added Q3: Si2305, transistor-small-signal:BSS84
- added Q4: BSS131, transistor-small-signal:BSS123
- added R5, R6: 100k, eagle-ltspice:RR1206
- PROG, RST: value (none) -> B3U-1000PB; device switch-omron:10-XX -> SnapEDA-Library2:B3U-1000PB
Connections:
- removed net DIO: SJ1.2, U1.IO26
- removed net N$7: LED_R.A, R23.2
- removed net N$8: LED_G.A, R25.2
- new net BUSY: U1.IO33, U3.DIO2
- new net DIO1: SJ1.3, U3.DIO1
- new net N$2: SJ1.2, U1.IO32
- new net N$3: LED_R.C, R23.1
- new net N$4: LED_G.C, R25.1
- new net N$9: Q3.G, Q4.D, R5.1
- new net PERIF: Q4.G, R6.2, U1.IO26
- net CMD_ALIM(SIM): now also U1.IO34; no longer U1.IO15
- net DHT: now also U1.IO20; no longer U1.IO32
- net DIO3: now also U1.IO12; no longer SJ1.3
- net EXT1: now also U1.IO14; no longer U1.IO12
- net EXT2: now also U1.IO35; no longer U1.IO20
- net GND: now also C7.2, C8.2, PROG.1, Q4.S, R23.2, R25.2, R6.1, RST.1; no longer JP5(SIM7000).1, JP5(SIM7000).6, LED_G.C, LED_R.C, PROG.P, PROG.P1, RST.P, RST.P1
- net IO0: now also PROG.2; no longer PROG.S, PROG.S1
- net IOPWRKEY(SIM): now also U1.IO4; no longer JP5(SIM7000).4, U1.IO27
- net IORX(SIM): no longer JP5(SIM7000).3
- net IOSLEEP(SIM): now also U1.IO25; no longer JP5(SIM7000).7, U1.IO13
- net IOTX(SIM): no longer JP5(SIM7000).2
- net LED_G: now also LED_G.A, U1.IO2; no longer R25.1, U1.IO25
- net LED_R: now also LED_R.A, U1.IO13; no longer R23.1, U1.IO33
- net LIGHT: now also U1.SENSOR_VN
- net RFM_RST: now also U1.IO27; no longer U1.IO14
- net RST: now also RST.2; no longer RST.S, RST.S1
- net V+: now also C7.1, C8.1, Q3.D; no longer C16.1, C17.1, U3.3.3V
- net V-VCC(SIM): no longer JP5(SIM7000).5
- net VCC: now also C16.1, C17.1, Q3.S, R5.2, U3.3.3V
Other:
- note added: "U3 replaced by LoRaCC68 (Nice RF) B3 = DIO0 = NC B5 = DIO4 = NC A7 = DIO5 = NC"
- moved on the sheet: LED_G, LED_R, R23, R25, SJ1
